File: circuit-design/circuit.kicad_pcb (KiCad board)
At the start: 2 copper layers, 75 x 60 mm, 11 parts, among them U1 TPS2553

Commit message: fixed drillholes and pins of USB-C adapter
Parts:
- C4: footprint Capacitor_THT:CP_Radial_D10.0mm_P2.50mm -> Capacitor_THT:CP_Radial_D10.0mm_P3.50mm
Routing:
- net GND: track 129.9 -> 131.3 mm
