File: circuit-design/circuit.kicad_sch (KiCad schematic)
At the start: 13 parts, among them U1 TPS2553

Commit message: fixed drillholes and pins of USB-C adapter
Parts:
- C4: footprint Capacitor_THT:CP_Radial_D10.0mm_P2.50mm -> Capacitor_THT:CP_Radial_D10.0mm_P3.50mm
Changed lines of the file:
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@@
 			)
 		)
-		(property "Footprint" "Capacitor_THT:CP_Radial_D10.0mm_P2.50mm"
+		(property "Footprint" "Capacitor_THT:CP_Radial_D10.0mm_P3.50mm"
 			(at 155.9052 95.25 0)
 			(effects
